File: kicad_project/esp8266-mitsubishi-cn105-pcb.kicad_pcb (KiCad board)
At the start: 2 copper layers, 60 x 30 mm, 30 parts, among them J1 S4B-PH-K-S, J2 Conn_01x06, J3 Conn_02x04_Odd_Even, Q1 BSS138, Q2 BSS138, SW1 SW_Push, SW2 SW_Push, U1 ESP-12F, U2 AP2112K-3.3

Commit message: Final production design
Parts:
- C4, C5: footprint Capacitor_SMD:C_0805_2012Metric_Pad1.18x1.45mm_HandSolder -> Capacitor_SMD:C_0603_1608Metric_Pad1.08x0.95mm_HandSolder
- R1, R2, R3, R4, R5, R6, R7, R8, R9: footprint Resistor_SMD:R_0805_2012Metric_Pad1.20x1.40mm_HandSolder -> Capacitor_SMD:C_0603_1608Metric_Pad1.08x0.95mm_HandSolder
Routing:
- net Net-(U1-GPIO15): track 7.08 -> 7.81 mm
