File: kicad_project/esp8266-mitsubishi-cn105-pcb.kicad_sch (KiCad schematic)
At the start: 0 parts

Commit message: Final (hopefully) production design
Parts:
- added C1, C2: 1uF, Capacitor_SMD:C_0805_2012Metric_Pad1.18x1.45mm_HandSolder, symbol Device:C
- added C3: 10uF, Capacitor_SMD:C_1206_3216Metric_Pad1.33x1.80mm_HandSolder, symbol Device:C
- added C4, C5: 0.1uF, Capacitor_SMD:C_0805_2012Metric_Pad1.18x1.45mm_HandSolder, symbol Device:C
- added H1, H2, H3, H4: MountingHole_Pad, MountingHole:MountingHole_3.2mm_M3_DIN965_Pad, symbol Mechanical:MountingHole_Pad
- added J1: S4B-PH-K-S, Connector_JST:JST_PH_S4B-PH-K_1x04_P2.00mm_Horizontal, symbol Connector_Generic:Conn_01x04
- added J2: Conn_01x06, Connector_PinHeader_2.54mm:PinHeader_1x06_P2.54mm_Vertical, symbol Connector_Generic:Conn_01x06
- added J3: Conn_02x04_Odd_Even, Connector_PinHeader_1.27mm:PinHeader_2x04_P1.27mm_Vertical, symbol Connector_Generic:Conn_02x04_Odd_Even
- added Q1, Q2: BSS138, Package_TO_SOT_SMD:SOT-23, symbol Transistor_FET:BSS138
- added R1, R2, R3, R4, R5, R6, R7, R8, R9: 10KOhm, Resistor_SMD:R_0805_2012Metric_Pad1.20x1.40mm_HandSolder, symbol Device:R
- added SW1, SW2: SW_Push, Button_Switch_SMD:SW_Tactile_SPST_NO_Straight_CK_PTS636Sx25SMTRLFS, symbol Switch:SW_Push
- added TP1, TP2, TP3: TestPoint, TestPoint:TestPoint_Pad_D2.0mm, symbol Connector:TestPoint
- added U1: ESP-12F, RF_Module:ESP-12E, symbol RF_Module:ESP-12F
- added U2: AP2112K-3.3, Package_TO_SOT_SMD:SOT-23-5, symbol Regulator_Linear:AP2112K-3.3
Connections:
- new net: R1.1, U1.3 (EN)
- new net: R3.2, U1.16 (GPIO15)
- new net: R2.2, U1.17 (GPIO2)
- new net +3.3V: C2.1, C3.1, C4.1, J2.4 (Pin_4), J3.3 (Pin_3), Q1.1 (G), Q2.1 (G), R1.2, R2.1, R4.1, R5.1, R6.1, R8.1, TP3.1, U1.8 (VCC), U2.5 (VOUT)
- new net +5V: C1.1, J1.2 (Pin_2), J3.2 (Pin_2), R7.1, R9.1, TP2.1, U2.1 (VIN), U2.3 (EN)
- new net AC_RX: J1.3 (Pin_3), Q1.3 (D), R7.2
- new net AC_TX: J1.4 (Pin_4), Q2.3 (D), R9.2
- new net ESP_RX: J2.3 (Pin_3), Q2.2 (S), R8.2, U1.21 (GPIO3/RXD)
- new net ESP_TX: J2.2 (Pin_2), Q1.2 (S), R6.2, U1.22 (GPIO1/TXD)
- new net GND: C1.2, C2.2, C3.2, C4.2, C5.1, J1.1 (Pin_1), J2.1 (Pin_1), J3.1 (Pin_1), R3.1, SW1.1, SW2.1, TP1.1, U1.15 (GND), U2.2 (GND)
- new net GPIO0: J2.6 (Pin_6), R5.2, SW2.2, U1.18 (GPIO0)
- new net GPIO12: J3.6 (Pin_6), U1.6 (GPIO12)
- new net GPIO13: J3.8 (Pin_8), U1.7 (GPIO13)
- new net GPIO14: J3.4 (Pin_4), U1.5 (GPIO14)
- new net GPIO4: J3.5 (Pin_5), U1.19 (GPIO4)
- new net GPIO5: J3.7 (Pin_7), U1.20 (GPIO5)
- new net ~{RST}: C5.2, J2.5 (Pin_5), R4.2, SW1.2, U1.1 (~{RST})
- no-connect marks 0 -> 11
Other:
- note added: "3.3V regulator"
- note added: "AC unit connector"
- note added: "Boot mode selection"
- note added: "FLASH"
- note added: "GPIO header"
- note added: "Headers"
- note added: "MCU"
- note added: "Programming header"
- note added: "RESET"
- note added: "UART level shifting"

Commit message: Final production design
Parts:
- C4, C5: footprint Capacitor_SMD:C_0805_2012Metric_Pad1.18x1.45mm_HandSolder -> Capacitor_SMD:C_0603_1608Metric_Pad1.08x0.95mm_HandSolder
- R1, R2, R3, R4, R5, R6, R7, R8, R9: footprint Resistor_SMD:R_0805_2012Metric_Pad1.20x1.40mm_HandSolder -> Capacitor_SMD:C_0603_1608Metric_Pad1.08x0.95mm_HandSolder
Changed lines of the file:
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@@
 			)
 		)
-		(property "Footprint" "Resistor_SMD:R_0805_2012Metric_Pad1.20x1.40mm_HandSolder"
+		(property "Footprint" "Capacitor_SMD:C_0603_1608Metric_Pad1.08x0.95mm_HandSolder"
 			(at 134.112 45.72 90)
 			(effects
@@
 			)
 		)
-		(property "Footprint" "Resistor_SMD:R_0805_2012Metric_Pad1.20x1.40mm_HandSolder"
+		(property "Footprint" "Capacitor_SMD:C_0603_1608Metric_Pad1.08x0.95mm_HandSolder"
 			(at 248.92 38.862 90)
 			(effects
@@
 			)
 		)
-		(property "Footprint" "Resistor_SMD:R_0805_2012Metric_Pad1.20x1.40mm_HandSolder"
+		(property "Footprint" "Capacitor_SMD:C_0603_1608Metric_Pad1.08x0.95mm_HandSolder"
 			(at 46.99 112.522 90)
 			(effects
@@
 			)
 		)
-		(property "Footprint" "Resistor_SMD:R_0805_2012Metric_Pad1.20x1.40mm_HandSolder"
+		(property "Footprint" "Capacitor_SMD:C_0603_1608Metric_Pad1.08x0.95mm_HandSolder"
 			(at 248.92 88.392 90)
 			(effects
@@
 			)
 		)
-		(property "Footprint" "Capacitor_SMD:C_0805_2012Metric_Pad1.18x1.45mm_HandSolder"
+		(property "Footprint" "Capacitor_SMD:C_0603_1608Metric_Pad1.08x0.95mm_HandSolder"
 			(at 49.2252 167.64 0)
 			(effects
@@
 			)
 		)
-		(property "Footprint" "Capacitor_SMD:C_0805_2012Metric_Pad1.18x1.45mm_HandSolder"
+		(property "Footprint" "Capacitor_SMD:C_0603_1608Metric_Pad1.08x0.95mm_HandSolder"
 			(at 133.35 59.9948 0)
 			(effects
@@
 			)
 		)
-		(property "Footprint" "Resistor_SMD:R_0805_2012Metric_Pad1.20x1.40mm_HandSolder"
+		(property "Footprint" "Capacitor_SMD:C_0603_1608Metric_Pad1.08x0.95mm_HandSolder"
 			(at 95.758 139.7 90)
 			(effects
@@
 			)
 		)
-		(property "Footprint" "Resistor_SMD:R_0805_2012Metric_Pad1.20x1.40mm_HandSolder"
+		(property "Footprint" "Capacitor_SMD:C_0603_1608Metric_Pad1.08x0.95mm_HandSolder"
 			(at 174.752 48.26 90)
 			(effects
@@
 			)
 		)
-		(property "Footprint" "Resistor_SMD:R_0805_2012Metric_Pad1.20x1.40mm_HandSolder"
+		(property "Footprint" "Capacitor_SMD:C_0603_1608Metric_Pad1.08x0.95mm_HandSolder"
 			(at 113.03 112.522 90)
 			(effects
@@
 			)
 		)
-		(property "Footprint" "Resistor_SMD:R_0805_2012Metric_Pad1.20x1.40mm_HandSolder"
+		(property "Footprint" "Capacitor_SMD:C_0603_1608Metric_Pad1.08x0.95mm_HandSolder"
 			(at 248.92 54.102 90)
 			(effects
@@
 			)
 		)
-		(property "Footprint" "Resistor_SMD:R_0805_2012Metric_Pad1.20x1.40mm_HandSolder"
+		(property "Footprint" "Capacitor_SMD:C_0603_1608Metric_Pad1.08x0.95mm_HandSolder"
 			(at 248.92 73.152 90)
 			(effects
